Commit message: slam_toolbox

File: src/bot_description/urdf/lidar.xacro (robot description, xacro)
@@ -43,5 +43,5 @@
             <plugin name="laser_controller" filename="libgazebo_ros_ray_sensor.so">
                 <ros>
-                    <argument>--ros-args --remap ~/out:=scan</argument>
+                    <argument>~/out:=scan</argument>
                 </ros>
                 <output_type>sensor_msgs/LaserScan</output_type>

File: src/bot_description/urdf/robot_core.xacro (robot description, xacro)
@@ -1,6 +1,16 @@
 <?xml version="1.0"?>
 <robot xmlns:xacro="http://www.ros.org/wiki/xacro">
+    <!-- BASE LINK -->
     <link name="base_link">
     </link>
+    <!-- BASE FOOTPRINT -->
+    <link name="base_footprint">
+    </link>
+    <joint name="base_footprint_joint" type="fixed">
+        <parent link="base_link" />
+        <child link="base_footprint" />
+        <origin xyz="0 0 0" />
+    </joint>
+    <!-- CHASSIS -->
     <joint name="chassis_joint" type="fixed">
         <parent link="base_link" />
